File: Hardware/Pre_Amp_8CH/Audio_Out.kicad_sch (KiCad schematic)
At the start: 0 parts

Commit message: RCA in & OUT
Parts:
- added J2: PJRAS4X2U01AUX, Pre_Amp_8CH_Footprints:PJRAS4X2U01AUX, symbol Pre_Amp_8CH_Symbols:PJRAS4X2U01AUX
Changed lines of the file:
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@@
 	(generator_version "9.0")
 	(paper "A4")
+	(symbol
+		(lib_id "Pre_Amp_8CH_Symbols:PJRAS4X2U01AUX")
+		(at 38.1 38.1 0)
+		(unit 1)
+		(exclude_from_sim no)
+		(in_bom yes)
+		(on_board yes)
+		(dnp no)
+		(property "Reference" "J2"
+			(at 39.37 35.052 0)
+			(effects
+				(font
+					(size 1.27 1.27)
+				)
+			)
+		)
+		(property "Value" "PJRAS4X2U01AUX"
+			(at 46.482 37.338 0)
+			(effects
+				(font
+					(size 1.27 1.27)
+				)
+			)
+		)
+		(property "Footprint" "Pre_Amp_8CH_Footprints:PJRAS4X2U01AUX"
+			(at 59.69 133.02 0)
+			(effects
+				(font
+					(size 1.27 1.27)
+				)
+				(justify left top)
+				(hide yes)
+			)
+		)
+		(property "Datasheet" "https://www.switchcraft.com/assets/1/24/pjras4x2u__x_series_cd.pdf?4683"
+			(at 59.69 233.02 0)
+			(effects
+				(font
+					(size 1.27 1.27)
+				)
+				(justify left top)
+				(hide yes)
+			)
+		)
+		(property "Description" "3.20mm ID, 9.00mm OD (RCA) Phono (RCA) Jack Mono Connector Solder"
+			(at 74.93 37.592 0)
+			(effects
+				(font
+					(size 1.27 1.27)
+				)
+				(hide yes)
+			)
+		)
+		(property "Height" "27"
+			(at 59.69 433.02 0)
+			(effects
+				(font
+					(size 1.27 1.27)
+				)
+				(justify left top)
+				(hide yes)
+			)
+		)
+		(property "Mouser Part Number" "502-PJRAS4X2U01AUX"
+			(at 59.69 533.02 0)
+			(effects
+				(font
+					(size 1.27 1.27)
+				)
+				(justify left top)
+				(hide yes)
+			)
+		)
+		(property "Mouser Price/Stock" "https://www.mouser.co.uk/ProductDetail/Switchcraft/PJRAS4X2U01AUX?qs=mcPJWgAPNrcm869EbXbltg%3D%3D"
+			(at 59.69 633.02 0)
+			(effects
+				(font
+					(size 1.27 1.27)
+				)
+				(justify left top)
+				(hide yes)
+			)
+		)
+		(property "Manufacturer_Name" "Switchcraft"
+			(at 59.69 733.02 0)
+			(effects
+				(font
+					(size 1.27 1.27)
+				)
+				(justify left top)
+				(hide yes)
+			)
+		)
+		(property "Manufacturer_Part_Number" "PJRAS4X2U01AUX"
+			(at 59.69 833.02 0)
+			(effects
+				(font
+					(size 1.27 1.27)
+				)
+				(justify left top)
+				(hide yes)
+			)
+		)
+		(pin "T11"
+		)
+		(pin "T21"
+		)
+		(pin "T22"
+		)
+		(pin "S2"
+		)
+		(pin "T31"
+		)
+		(pin "S3"
+		)
+		(pin "T41"
+		)
+		(pin "T32"
+		)
+		(pin "S4"
+		)
+		(pin "T12"
+		)
+		(pin "S1"
+		)
+		(pin "T42"
+		)
+		(instances
+			(project "Pre_Amp_8CH"
+				(path "/95391f5e-c27a-414f-9293-205fef445dea/45d7762c-a846-43dd-9c78-69cecc0e82eb"
+					(reference "J2")
+					(unit 1)
+				)
+			)
+		)
+	)
 )

Commit message: DSP start
Parts:
- renumbered J2 to J401
Changed lines of the file:
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@@
 		(on_board yes)
 		(dnp no)
-		(property "Reference" "J2"
+		(property "Reference" "J401"
 			(at 39.37 35.052 0)
 			(effects
@@
 			(project "Pre_Amp_8CH"
 				(path "/95391f5e-c27a-414f-9293-205fef445dea/45d7762c-a846-43dd-9c78-69cecc0e82eb"
-					(reference "J2")
+					(reference "J401")
 					(unit 1)
 				)
