File: Hardware/Pre_Amp_8CH/Controller.kicad_sch (KiCad schematic)
At the start: 0 parts

Commit message: DSP start
Parts:
- added U601: STM32F410R8Tx, Package_QFP:LQFP-64_10x10mm_P0.5mm, symbol MCU_ST_STM32F4:STM32F410R8Tx
Connections:
- new net: U601.18 (VSS), U601.31 (VSS), U601.47 (VSS), U601.63 (VSS)
