File: Hardware/Pre_Amp_8CH/Audio_DSP.kicad_sch (KiCad schematic)
At the start: 0 parts

Commit message: DSP start
Parts:
- added C501, C503, C504, C505, C506, C507, C510, C513: 100nF, Capacitor_SMD:C_0805_2012Metric_Pad1.18x1.45mm_HandSolder, symbol Device:C
- added C502: 1nF, Capacitor_SMD:C_0805_2012Metric_Pad1.18x1.45mm_HandSolder, symbol Device:C
- added C508: 1n2, Capacitor_SMD:C_0805_2012Metric_Pad1.18x1.45mm_HandSolder, symbol Device:C
- added C509: 2u2, Capacitor_SMD:C_0805_2012Metric_Pad1.18x1.45mm_HandSolder, symbol Device:C
- added C511, C512: 100p, Capacitor_SMD:C_0805_2012Metric_Pad1.18x1.45mm_HandSolder, symbol Device:C
- added C514: 47p, Capacitor_SMD:C_0805_2012Metric_Pad1.18x1.45mm_HandSolder, symbol Device:C
- added FB501: 600ohm100MHz, Resistor_SMD:R_0805_2012Metric_Pad1.20x1.40mm_HandSolder, symbol Device:FerriteBead_Small
- added IC501: STA309A13TR, Pre_Amp_8CH_Footprints:QFP50P1200X1200X160-64N, symbol Pre_Amp_8CH_Symbols:STA309A13TR
- added R501: 3K4, Resistor_SMD:R_0805_2012Metric_Pad1.20x1.40mm_HandSolder, symbol Device:R
- added R502, R503: 10K, Resistor_SMD:R_0805_2012Metric_Pad1.20x1.40mm_HandSolder, symbol Device:R
Connections:
- new net: C508.1, C511.1, R501.2
- new net: C513.1, IC501.24 (VDDA)
- new net +3V3: C501.1, C503.1, C504.1, C505.1, C506.1, C507.1, C509.1, C510.1, IC501.1 (MVO), IC501.12 (VDD_2), IC501.28 (VDD_3), IC501.3 (VDD_1), IC501.35 (VDD_4), IC501.44 (VDD_5), IC501.52 (VDD_6), IC501.59 (VDD_7), R502.1, R503.1
- new net BICKI: IC501.11 (BICKI)
- new net BICKO: IC501.55 (BICKO)
- new net GNDD: C501.2, C502.2, C503.2, C504.2, C505.2, C506.2, C507.2, C509.2, C510.2, C513.2, C514.2, FB501.2, IC501.13 (GND_3), IC501.17 (SA), IC501.2 (GND_1), IC501.27 (GND_4), IC501.36 (GND_5), IC501.4 (GND_2), IC501.45 (GND_6), IC501.53 (GND_7), IC501.60 (GND_8)
- new net I2C_SCL: IC501.19 (SCL), R503.2
- new net I2C_SDA: IC501.18 (SDA), R502.2
- new net LRCKI: C514.1, IC501.10 (LRCKI)
- new net LRCKO: IC501.56 (LRCKO)
- new net MCLK: IC501.20 (XTI)
- new net PLL-Filter: C512.1, IC501.21 (FILTER_PLL), R501.1
- new net PLL-Filter-GND: C508.2, C511.2, C512.2, FB501.1, IC501.23 (GNDA)
- new net POWER_ON_RESET: C502.1, IC501.15 (RESET)
- new net SDATA_IN_12: IC501.9 (SDI_12)
- new net SDATA_IN_34: IC501.8 (SDI_34)
- new net SDATA_IN_56: IC501.7 (SDI_56)
- new net SDATA_IN_78: IC501.6 (SDI_78)
- new net SDATA_OUT_12: IC501.57 (SDO_12)
- new net SDATA_OUT_34: IC501.58 (SDO_34)
- new net SDATA_OUT_56: IC501.62 (SDO_56)
- new net SDATA_OUT_78: IC501.63 (SDO_78)
- no-connect marks 0 -> 12
Other:
- note added: "Decoupling"
- note added: "I2S IN"
- note added: "PLL-Filter"

Commit message: PSU
Parts:
- added C515: 1nF, Capacitor_SMD:C_0603_1608Metric_Pad1.08x0.95mm_HandSolder, symbol Device:C
- C501, C502, C503, C504, C505, C506, C507, C508, C510, C511, C512, C513, C514: footprint Capacitor_SMD:C_0805_2012Metric_Pad1.18x1.45mm_HandSolder -> Capacitor_SMD:C_0603_1608Metric_Pad1.08x0.95mm_HandSolder
- R501, R502, R503: footprint Resistor_SMD:R_0805_2012Metric_Pad1.20x1.40mm_HandSolder -> Resistor_SMD:R_0603_1608Metric_Pad0.98x0.95mm_HandSolder
Connections:
- net GNDD: now also IC501.16 (PLLB), C515.2
- net CKOUT: now reaches IC501.25 (CKOUT)
- net OUT8_B: now reaches IC501.29 (OUT8_B)
- net OUT8_A: now reaches IC501.30 (OUT8_A)
- net OUT7_B: now reaches IC501.31 (OUT7_B)
- net OUT7_A: now reaches IC501.32 (OUT7_A)
- net OUT6_B: now reaches IC501.33 (OUT6_B)
- net OUT6_A: now reaches IC501.34 (OUT6_A)
- net OUT5_B: now reaches IC501.38 (OUT5_B)
- net OUT5_A: now reaches IC501.39 (OUT5_A)
- net OUT4_B: now reaches IC501.40 (OUT4_B)
- net OUT4_A: now reaches IC501.41 (OUT4_A)
- net OUT3_B: now reaches IC501.42 (OUT3_B)
- net OUT3_A: now reaches IC501.43 (OUT3_A)
- net OUT2_B: now reaches IC501.47 (OUT2_B)
- net OUT2_A: now reaches IC501.48 (OUT2_A)
- net OUT1_B: now reaches IC501.49 (OUT1_B)
- net OUT1_A: now reaches IC501.50 (OUT1_A)
- net EAPD: now reaches IC501.51 (EAPD)
- net PWDN: now reaches IC501.64 (PWDN)
- net PWDN: now also C515.1
- no-connect marks 12 -> 29
