File: Hardware/Pre_Amp_8CH/PSU.kicad_sch (KiCad schematic)
At the start: 0 parts

Commit message: RCA in & OUT
Parts:
- added J3: USB_C_Receptacle_PowerOnly_6P, Connector_USB:USB_C_Receptacle_GCT_USB4125-xx-x-0190_6P_TopMnt_Horizontal, symbol Connector:USB_C_Receptacle_PowerOnly_6P
- added R1, R2: 5K1, Resistor_SMD:R_0805_2012Metric_Pad1.20x1.40mm_HandSolder, symbol Device:R
Connections:
- new net CC1: J3.A5 (CC1), R2.1
- new net CC2: J3.B5 (CC2), R1.1
- new net GNDD: J3.A12 (GND), J3.B12 (GND), J3.S1 (SHIELD), R1.2, R2.2
- new net VBUS: J3.A9 (VBUS), J3.B9 (VBUS)

Commit message: DSP start
Parts:
- renumbered J3 to J201, R1 to R201, R2 to R202
Changed lines of the file:
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@@
 		(dnp no)
 		(fields_autoplaced yes)
-		(property "Reference" "R2"
+		(property "Reference" "R202"
 			(at 91.44 66.0399 0)
 			(effects
@@
 			(project "Pre_Amp_8CH"
 				(path "/95391f5e-c27a-414f-9293-205fef445dea/a5767999-db98-4724-8c72-273c259d6263"
-					(reference "R2")
+					(reference "R202")
 					(unit 1)
 				)
@@
 		(dnp no)
 		(fields_autoplaced yes)
-		(property "Reference" "J3"
+		(property "Reference" "J201"
 			(at 48.26 33.02 0)
 			(effects
@@
 			(project ""
 				(path "/95391f5e-c27a-414f-9293-205fef445dea/a5767999-db98-4724-8c72-273c259d6263"
-					(reference "J3")
+					(reference "J201")
 					(unit 1)
 				)
@@
 		(dnp no)
 		(fields_autoplaced yes)
-		(property "Reference" "#PWR06"
+		(property "Reference" "#PWR0202"
 			(at 48.26 82.55 0)
 			(effects
@@
 			(project "Pre_Amp_8CH"
 				(path "/95391f5e-c27a-414f-9293-205fef445dea/a5767999-db98-4724-8c72-273c259d6263"
-					(reference "#PWR06")
+					(reference "#PWR0202")
 					(unit 1)
 				)
@@
 		(dnp no)
 		(fields_autoplaced yes)
-		(property "Reference" "R1"
+		(property "Reference" "R201"
 			(at 78.74 66.0399 0)
 			(effects
@@
 			(project ""
 				(path "/95391f5e-c27a-414f-9293-205fef445dea/a5767999-db98-4724-8c72-273c259d6263"
-					(reference "R1")
+					(reference "R201")
 					(unit 1)
 				)
@@
 		(dnp no)
 		(fields_autoplaced yes)
-		(property "Reference" "#PWR08"
+		(property "Reference" "#PWR0204"
 			(at 88.9 82.55 0)
 			(effects
@@
 			(project "Pre_Amp_8CH"
 				(path "/95391f5e-c27a-414f-9293-205fef445dea/a5767999-db98-4724-8c72-273c259d6263"
-					(reference "#PWR08")
+					(reference "#PWR0204")
 					(unit 1)
 				)
@@
 		(dnp no)
 		(fields_autoplaced yes)
-		(property "Reference" "#PWR07"
+		(property "Reference" "#PWR0203"
 			(at 76.2 82.55 0)
 			(effects
@@
 			(project "Pre_Amp_8CH"
 				(path "/95391f5e-c27a-414f-9293-205fef445dea/a5767999-db98-4724-8c72-273c259d6263"
-					(reference "#PWR07")
+					(reference "#PWR0203")
 					(unit 1)
 				)
@@
 		(dnp no)
 		(fields_autoplaced yes)
-		(property "Reference" "#PWR05"
+		(property "Reference" "#PWR0201"
 			(at 40.64 82.55 0)
 			(effects
@@
 			(project ""
 				(path "/95391f5e-c27a-414f-9293-205fef445dea/a5767999-db98-4724-8c72-273c259d6263"
-					(reference "#PWR05")
-					(unit 1)
-				)
+					(reference "#PWR0201")
+					(unit 1)
+				)

Commit message: PSU
Parts:
- added C201, C202: 865060240001, Pre_Amp_8CH_Footprints:CP_Wurth_WCAP-ASLL-D4L5.5, symbol Pre_Amp_8CH_Symbols:865060240001
- added JP201: USB_jumper, Jumper:SolderJumper-2_P1.3mm_Open_Pad1.0x1.5mm, symbol Jumper:SolderJumper_2_Open
- added JP202: 3V3_jumper, Jumper:SolderJumper-2_P1.3mm_Open_Pad1.0x1.5mm, symbol Jumper:SolderJumper_2_Open
- added L201: BMRA000606301R0MA1, Pre_Amp_8CH_Footprints:INDPM7366X300N, symbol Pre_Amp_8CH_Symbols:BMRA000606301R0MA1
- added R203: 453k, Resistor_SMD:R_0603_1608Metric_Pad0.98x0.95mm_HandSolder, symbol Device:R
- added R204: 100k, Resistor_SMD:R_0603_1608Metric_Pad0.98x0.95mm_HandSolder, symbol Device:R
- added TP201: USB, TestPoint:TestPoint_Pad_D1.0mm, symbol Connector:TestPoint_Probe
- added TP202: 3V3, TestPoint:TestPoint_Pad_D1.0mm, symbol Connector:TestPoint_Probe
- added U201: TLV62569ADRL, Package_TO_SOT_SMD:SOT-563, symbol Regulator_Switching:TLV62569ADRL
- R201, R202: footprint Resistor_SMD:R_0805_2012Metric_Pad1.20x1.40mm_HandSolder -> Resistor_SMD:R_0603_1608Metric_Pad0.98x0.95mm_HandSolder
Connections:
- net GNDD: now also C201.2, C202.2, R204.2, U201.2 (GND)
- net VBUS: now also JP201.1 (A), TP201.1
- new net +3V3: JP202.2 (B)
- new net +5V: C201.1, JP201.2 (B), U201.3 (VIN), U201.5 (EN)
- new net 3V3_sb: C202.1, JP202.1 (A), L201.2, R203.1, TP202.1
- new net FB: R203.2, R204.1, U201.1 (FB)
- new net SW: L201.1, U201.4 (SW)
Other:
- note added: "1.14MHz"
- moved on the sheet: J201, R201, R202
